Commit message: add joints

File: src/rrbot/urdf/rrbot.xacro (robot description, xacro)
@@ -174,3 +174,19 @@
       </hardware>
     </ros2_control>
+  <joint name="left_wheel_joint">
+        <command_interface name="velocity">
+            <param name="min">-10</param>
+            <param name="max">10</param>
+        </command_interface>
+        <state_interface name="velocity"/>
+        <state_interface name="position"/>
+    </joint>
+    <joint name="right_wheel_joint">
+        <command_interface name="velocity">
+            <param name="min">-10</param>
+            <param name="max">10</param>
+        </command_interface>
+        <state_interface name="velocity"/>
+        <state_interface name="position"/>
+    </joint>
 </robot>
